File: pcb/dcc.kicad_sch (KiCad schematic)
At the start: 68 parts, among them U10 LM339, U11 LM339, U4 L78L05_SOT89, U5 L79L05_SOT89, U6 LM339, U7 LM339, U8 LM339, U9 4052

Commit message: Added values schottky.
Parts:
- D11, D12, D13, D14, D15, D16, D17, D18, D19, D20, D21, D22, D23, D24, D25, D26: value D_Schottky -> SS34; footprint (none) -> Diode_SMD:D_SMA_Handsoldering
Changed lines of the file:
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@@
       (effects (font (size 1.27 1.27)))
     )
-    (property "Value" "D_Schottky" (at 27.94 107.95 0)
-      (effects (font (size 1.27 1.27)) hide)
-    )
-    (property "Footprint" "" (at 39.37 109.22 0)
+    (property "Value" "SS34" (at 27.94 107.95 0)
+      (effects (font (size 1.27 1.27)) hide)
+    )
+    (property "Footprint" "Diode_SMD:D_SMA_Handsoldering" (at 39.37 109.22 0)
       (effects (font (size 1.27 1.27)) hide)
     )
@@
       (effects (font (size 1.27 1.27)))
     )
-    (property "Value" "D_Schottky" (at 248.285 82.55 0)
-      (effects (font (size 1.27 1.27)) hide)
-    )
-    (property "Footprint" "" (at 259.715 83.82 0)
+    (property "Value" "SS34" (at 248.285 82.55 0)
+      (effects (font (size 1.27 1.27)) hide)
+    )
+    (property "Footprint" "Diode_SMD:D_SMA_Handsoldering" (at 259.715 83.82 0)
       (effects (font (size 1.27 1.27)) hide)
     )
@@
       (effects (font (size 1.27 1.27)))
     )
-    (property "Value" "D_Schottky" (at 39.0525 59.69 0)
-      (effects (font (size 1.27 1.27)) hide)
-    )
-    (property "Footprint" "" (at 39.37 62.865 0)
+    (property "Value" "SS34" (at 39.0525 59.69 0)
+      (effects (font (size 1.27 1.27)) hide)
+    )
+    (property "Footprint" "Diode_SMD:D_SMA_Handsoldering" (at 39.37 62.865 0)
       (effects (font (size 1.27 1.27)) hide)
     )
@@
       (effects (font (size 1.27 1.27)))
     )
-    (property "Value" "D_Schottky" (at 248.285 57.15 0)
-      (effects (font (size 1.27 1.27)) hide)
-    )
-    (property "Footprint" "" (at 259.715 58.42 0)
+    (property "Value" "SS34" (at 248.285 57.15 0)
+      (effects (font (size 1.27 1.27)) hide)
+    )
+    (property "Footprint" "Diode_SMD:D_SMA_Handsoldering" (at 259.715 58.42 0)
       (effects (font (size 1.27 1.27)) hide)
     )
@@
       (effects (font (size 1.27 1.27)))
     )
-    (property "Value" "D_Schottky" (at 39.0525 110.49 0)
-      (effects (font (size 1.27 1.27)) hide)
-    )
-    (property "Footprint" "" (at 39.37 113.665 0)
+    (property "Value" "SS34" (at 39.0525 110.49 0)
+      (effects (font (size 1.27 1.27)) hide)
+    )
+    (property "Footprint" "Diode_SMD:D_SMA_Handsoldering" (at 39.37 113.665 0)
       (effects (font (size 1.27 1.27)) hide)
     )
@@
       (effects (font (size 1.27 1.27)))
     )
-    (property "Value" "D_Schottky" (at 259.3975 34.29 0)
-      (effects (font (size 1.27 1.27)) hide)
-    )
-    (property "Footprint" "" (at 259.715 37.465 0)
+    (property "Value" "SS34" (at 259.3975 34.29 0)
+      (effects (font (size 1.27 1.27)) hide)
+    )
+    (property "Footprint" "Diode_SMD:D_SMA_Handsoldering" (at 259.715 37.465 0)
       (effects (font (size 1.27 1.27)) hide)
     )
@@
       (effects (font (size 1.27 1.27)))
     )
-    (property "Value" "D_Schottky" (at 39.0525 85.09 0)
-      (effects (font (size 1.27 1.27)) hide)
-    )
-    (property "Footprint" "" (at 39.37 88.265 0)
+    (property "Value" "SS34" (at 39.0525 85.09 0)
+      (effects (font (size 1.27 1.27)) hide)
+    )
+    (property "Footprint" "Diode_SMD:D_SMA_Handsoldering" (at 39.37 88.265 0)
       (effects (font (size 1.27 1.27)) hide)
     )
@@
       (effects (font (size 1.27 1.27)))
     )
-    (property "Value" "D_Schottky" (at 27.94 82.55 0)
-      (effects (font (size 1.27 1.27)) hide)
-    )
-    (property "Footprint" "" (at 39.37 83.82 0)
+    (property "Value" "SS34" (at 27.94 82.55 0)
+      (effects (font (size 1.27 1.27)) hide)
+    )
+    (property "Footprint" "Diode_SMD:D_SMA_Handsoldering" (at 39.37 83.82 0)
       (effects (font (size 1.27 1.27)) hide)
     )
@@
       (effects (font (size 1.27 1.27)))
     )
-    (property "Value" "D_Schottky" (at 259.3975 59.69 0)
-      (effects (font (size 1.27 1.27)) hide)
-    )
-    (property "Footprint" "" (at 259.715 62.865 0)
+    (property "Value" "SS34" (at 259.3975 59.69 0)
+      (effects (font (size 1.27 1.27)) hide)
+    )
+    (property "Footprint" "Diode_SMD:D_SMA_Handsoldering" (at 259.715 62.865 0)
       (effects (font (size 1.27 1.27)) hide)
     )
@@
       (effects (font (size 1.27 1.27)))
     )
-    (property "Value" "D_Schottky" (at 39.0525 34.29 0)
-      (effects (font (size 1.27 1.27)) hide)
-    )
-    (property "Footprint" "" (at 39.37 37.465 0)
+    (property "Value" "SS34" (at 39.0525 34.29 0)
+      (effects (font (size 1.27 1.27)) hide)
+    )
+    (property "Footprint" "Diode_SMD:D_SMA_Handsoldering" (at 39.37 37.465 0)
       (effects (font (size 1.27 1.27)) hide)
     )
@@
       (effects (font (size 1.27 1.27)))
     )
-    (property "Value" "D_Schottky" (at 248.285 31.75 0)
-      (effects (font (size 1.27 1.27)) hide)
-    )
-    (property "Footprint" "" (at 259.715 33.02 0)
+    (property "Value" "SS34" (at 248.285 31.75 0)
+      (effects (font (size 1.27 1.27)) hide)
+    )
+    (property "Footprint" "Diode_SMD:D_SMA_Handsoldering" (at 259.715 33.02 0)
       (effects (font (size 1.27 1.27)) hide)
     )
@@
       (effects (font (size 1.27 1.27)))
     )
-    (property "Value" "D_Schottky" (at 260.0325 107.315 0)
-      (effects (font (size 1.27 1.27)) hide)
-    )
-    (property "Footprint" "" (at 260.35 110.49 0)
+    (property "Value" "SS34" (at 260.0325 107.315 0)
+      (effects (font (size 1.27 1.27)) hide)
+    )
+    (property "Footprint" "Diode_SMD:D_SMA_Handsoldering" (at 260.35 110.49 0)
       (effects (font (size 1.27 1.27)) hide)
     )
@@
       (effects (font (size 1.27 1.27)))
     )
-    (property "Value" "D_Schottky" (at 27.94 31.75 0)
-      (effects (font (size 1.27 1.27)) hide)
-    )
-    (property "Footprint" "" (at 39.37 33.02 0)
+    (property "Value" "SS34" (at 27.94 31.75 0)
+      (effects (font (size 1.27 1.27)) hide)
+    )
+    (property "Footprint" "Diode_SMD:D_SMA_Handsoldering" (at 39.37 33.02 0)
       (effects (font (size 1.27 1.27)) hide)
     )
@@
       (effects (font (size 1.27 1.27)))
     )
-    (property "Value" "D_Schottky" (at 248.92 104.775 0)
-      (effects (font (size 1.27 1.27)) hide)
-    )
-    (property "Footprint" "" (at 260.35 106.045 0)
+    (property "Value" "SS34" (at 248.92 104.775 0)
+      (effects (font (size 1.27 1.27)) hide)
+    )
+    (property "Footprint" "Diode_SMD:D_SMA_Handsoldering" (at 260.35 106.045 0)
       (effects (font (size 1.27 1.27)) hide)
     )
@@
       (effects (font (size 1.27 1.27)))
     )
-    (property "Value" "D_Schottky" (at 259.3975 85.09 0)
-      (effects (font (size 1.27 1.27)) hide)
-    )
-    (property "Footprint" "" (at 259.715 88.265 0)
+    (property "Value" "SS34" (at 259.3975 85.09 0)
+      (effects (font (size 1.27 1.27)) hide)
+    )
+    (property "Footprint" "Diode_SMD:D_SMA_Handsoldering" (at 259.715 88.265 0)
       (effects (font (size 1.27 1.27)) hide)
     )
@@
       (effects (font (size 1.27 1.27)))
     )
-    (property "Value" "D_Schottky" (at 27.94 57.15 0)
-      (effects (font (size 1.27 1.27)) hide)
-    )
-    (property "Footprint" "" (at 39.37 58.42 0)
-      (effects (font (size 1.27 1.27)) hide)
-    )
+    (property "Value" "SS34" (at 27.94 57.15 0)
+      (effects (font (size 1.27 1.27)) hide)
+    )
+    (property "Footprint" "Diode_SMD:D_SMA_Handsoldering" (at 39.37 58.42 0)
+      (effects (font (size 1.27 1.27)) hide)
+    )
