File: pcb/railcomdet.kicad_sch (KiCad schematic)
At the start: 43 parts, among them J1 MVE252-5-V, J10 MVE252-5-V, J2 MVE252-5-V, J3 MVE252-5-V, J7 MVE252-5-V, J8 MVE252-5-V, J9 MVE252-5-V, U1 VO0631T, U2 VO0631T, U3 VO0631T

Commit message: Add several notes.
Other:
- note added: "Place near U1"
- note added: "Place near U2 & U3."
- moved on the sheet: C2, C3
Changed lines of the file:
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@@
     (stroke (width 0) (type default))
   )
-  (wire (pts (xy 184.15 21.59) (xy 184.15 22.86))
+  (wire (pts (xy 193.04 21.59) (xy 193.04 22.86))
     (stroke (width 0) (type default))
   )
@@
     (stroke (width 0) (type default))
   )
-  (wire (pts (xy 170.18 21.59) (xy 170.18 22.86))
+  (wire (pts (xy 179.07 21.59) (xy 179.07 22.86))
     (stroke (width 0) (type default))
   )
@@
     (stroke (width 0) (type default))
   )
-  (wire (pts (xy 170.18 31.75) (xy 170.18 30.48))
+  (wire (pts (xy 179.07 31.75) (xy 179.07 30.48))
     (stroke (width 0) (type default))
   )
@@
     (stroke (width 0) (type default))
   )
-  (wire (pts (xy 184.15 31.75) (xy 184.15 30.48))
+  (wire (pts (xy 193.04 31.75) (xy 193.04 30.48))
     (stroke (width 0) (type default))
   )
@@
   (wire (pts (xy 153.67 149.86) (xy 170.18 149.86))
     (stroke (width 0) (type default))
+  )
+  (text "Place near U2 & U3." (at 152.4 27.305 0)
+    (effects (font (size 1.27 1.27)) (justify left bottom))
+  )
+  (text "Place near U1" (at 112.395 27.305 0)
+    (effects (font (size 1.27 1.27)) (justify left bottom))
   )
   (label "GND" (at 252.095 33.655 0) (fields_autoplaced)
@@
     )
   )
-  (symbol (lib_id "Device:C") (at 184.15 26.67 0) (unit 1)
-    (in_bom yes) (on_board yes) (dnp no) (fields_autoplaced)
-    (property "Reference" "C3" (at 187.96 25.4 0)
-      (effects (font (size 1.27 1.27)) (justify left))
-    )
-    (property "Value" "100n" (at 187.96 27.94 0)
-      (effects (font (size 1.27 1.27)) (justify left))
-    )
-    (property "Footprint" "Capacitor_SMD:C_0805_2012Metric" (at 185.1152 30.48 0)
-      (effects (font (size 1.27 1.27)) hide)
-    )
-    (property "Datasheet" "~" (at 184.15 26.67 0)
+  (symbol (lib_id "Device:C") (at 193.04 26.67 0) (unit 1)
+    (in_bom yes) (on_board yes) (dnp no) (fields_autoplaced)
+    (property "Reference" "C3" (at 196.85 25.4 0)
+      (effects (font (size 1.27 1.27)) (justify left))
+    )
+    (property "Value" "100n" (at 196.85 27.94 0)
+      (effects (font (size 1.27 1.27)) (justify left))
+    )
+    (property "Footprint" "Capacitor_SMD:C_0805_2012Metric" (at 194.0052 30.48 0)
+      (effects (font (size 1.27 1.27)) hide)
+    )
+    (property "Datasheet" "~" (at 193.04 26.67 0)
       (effects (font (size 1.27 1.27)) hide)
     )
@@
     )
   )
-  (symbol (lib_id "power:+5V") (at 184.15 21.59 0) (unit 1)
-    (in_bom yes) (on_board yes) (dnp no) (fields_autoplaced)
-    (property "Reference" "#PWR019" (at 184.15 25.4 0)
-      (effects (font (size 1.27 1.27)) hide)
-    )
-    (property "Value" "+5V" (at 184.15 16.51 0)
-      (effects (font (size 1.27 1.27)))
-    )
-    (property "Footprint" "" (at 184.15 21.59 0)
-      (effects (font (size 1.27 1.27)) hide)
-    )
-    (property "Datasheet" "" (at 184.15 21.59 0)
+  (symbol (lib_id "power:+5V") (at 193.04 21.59 0) (unit 1)
+    (in_bom yes) (on_board yes) (dnp no) (fields_autoplaced)
+    (property "Reference" "#PWR019" (at 193.04 25.4 0)
+      (effects (font (size 1.27 1.27)) hide)
+    )
+    (property "Value" "+5V" (at 193.04 16.51 0)
+      (effects (font (size 1.27 1.27)))
+    )
+    (property "Footprint" "" (at 193.04 21.59 0)
+      (effects (font (size 1.27 1.27)) hide)
+    )
+    (property "Datasheet" "" (at 193.04 21.59 0)
       (effects (font (size 1.27 1.27)) hide)
     )
@@
     )
   )
-  (symbol (lib_id "power:GND") (at 184.15 31.75 0) (unit 1)
-    (in_bom yes) (on_board yes) (dnp no) (fields_autoplaced)
-    (property "Reference" "#PWR020" (at 184.15 38.1 0)
-      (effects (font (size 1.27 1.27)) hide)
-    )
-    (property "Value" "GND" (at 184.15 36.83 0)
-      (effects (font (size 1.27 1.27)))
-    )
-    (property "Footprint" "" (at 184.15 31.75 0)
-      (effects (font (size 1.27 1.27)) hide)
-    )
-    (property "Datasheet" "" (at 184.15 31.75 0)
+  (symbol (lib_id "power:GND") (at 193.04 31.75 0) (unit 1)
+    (in_bom yes) (on_board yes) (dnp no) (fields_autoplaced)
+    (property "Reference" "#PWR020" (at 193.04 38.1 0)
+      (effects (font (size 1.27 1.27)) hide)
+    )
+    (property "Value" "GND" (at 193.04 36.83 0)
+      (effects (font (size 1.27 1.27)))
+    )
+    (property "Footprint" "" (at 193.04 31.75 0)
+      (effects (font (size 1.27 1.27)) hide)
+    )
+    (property "Datasheet" "" (at 193.04 31.75 0)
       (effects (font (size 1.27 1.27)) hide)
     )
@@
     )
   )
-  (symbol (lib_id "Device:C") (at 170.18 26.67 0) (unit 1)
-    (in_bom yes) (on_board yes) (dnp no)
-    (property "Reference" "C2" (at 173.99 25.4 0)
-      (effects (font (size 1.27 1.27)) (justify left))
-    )
-    (property "Value" "100n" (at 173.99 27.94 0)
-      (effects (font (size 1.27 1.27)) (justify left))
-    )
-    (property "Footprint" "Capacitor_SMD:C_0805_2012Metric" (at 171.1452 30.48 0)
-      (effects (font (size 1.27 1.27)) hide)
-    )
-    (property "Datasheet" "~" (at 170.18 26.67 0)
+  (symbol (lib_id "Device:C") (at 179.07 26.67 0) (unit 1)
+    (in_bom yes) (on_board yes) (dnp no)
+    (property "Reference" "C2" (at 182.88 25.4 0)
+      (effects (font (size 1.27 1.27)) (justify left))
+    )
+    (property "Value" "100n" (at 182.88 27.94 0)
+      (effects (font (size 1.27 1.27)) (justify left))
+    )
+    (property "Footprint" "Capacitor_SMD:C_0805_2012Metric" (at 180.0352 30.48 0)
+      (effects (font (size 1.27 1.27)) hide)
+    )
+    (property "Datasheet" "~" (at 179.07 26.67 0)
       (effects (font (size 1.27 1.27)) hide)
     )
@@
     )
   )
-  (symbol (lib_id "power:GND") (at 170.18 31.75 0) (unit 1)
-    (in_bom yes) (on_board yes) (dnp no) (fields_autoplaced)
-    (property "Reference" "#PWR016" (at 170.18 38.1 0)
-      (effects (font (size 1.27 1.27)) hide)
-    )
-    (property "Value" "GND" (at 170.18 36.83 0)
-      (effects (font (size 1.27 1.27)))
-    )
-    (property "Footprint" "" (at 170.18 31.75 0)
-      (effects (font (size 1.27 1.27)) hide)
-    )
-    (property "Datasheet" "" (at 170.18 31.75 0)
+  (symbol (lib_id "power:GND") (at 179.07 31.75 0) (unit 1)
+    (in_bom yes) (on_board yes) (dnp no) (fields_autoplaced)
+    (property "Reference" "#PWR016" (at 179.07 38.1 0)
+      (effects (font (size 1.27 1.27)) hide)
+    )
+    (property "Value" "GND" (at 179.07 36.83 0)
+      (effects (font (size 1.27 1.27)))
+    )
+    (property "Footprint" "" (at 179.07 31.75 0)
+      (effects (font (size 1.27 1.27)) hide)
+    )
+    (property "Datasheet" "" (at 179.07 31.75 0)
       (effects (font (size 1.27 1.27)) hide)
     )
@@
     )
   )
-  (symbol (lib_id "power:+5V") (at 170.18 21.59 0) (unit 1)
-    (in_bom yes) (on_board yes) (dnp no) (fields_autoplaced)
-    (property "Reference" "#PWR015" (at 170.18 25.4 0)
-      (effects (font (size 1.27 1.27)) hide)
-    )
-    (property "Value" "+5V" (at 170.18 16.51 0)
-      (effects (font (size 1.27 1.27)))
-    )
-    (property "Footprint" "" (at 170.18 21.59 0)
-      (effects (font (size 1.27 1.27)) hide)
-    )
-    (property "Datasheet" "" (at 170.18 21.59 0)
+  (symbol (lib_id "power:+5V") (at 179.07 21.59 0) (unit 1)
+    (in_bom yes) (on_board yes) (dnp no) (fields_autoplaced)
+    (property "Reference" "#PWR015" (at 179.07 25.4 0)
+      (effects (font (size 1.27 1.27)) hide)
+    )
+    (property "Value" "+5V" (at 179.07 16.51 0)
+      (effects (font (size 1.27 1.27)))
+    )
+    (property "Footprint" "" (at 179.07 21.59 0)
+      (effects (font (size 1.27 1.27)) hide)
+    )
+    (property "Datasheet" "" (at 179.07 21.59 0)
       (effects (font (size 1.27 1.27)) hide)
     )
@@
   )
   (symbol (lib_id "Device:R") (at 180.34 139.7 90) (mirror x) (unit 1)
-    (in_bom yes) (on_board yes) (dnp no) (fields_autoplaced)
-    (property "Reference" "R12" (at 180.34 133.35 90)
-      (effects (font (size 1.27 1.27)))
-    )
-    (property "Value" "1k" (at 180.34 135.89 90)
-      (effects (font (size 1.27 1.27)))
-    )
+    (in_bom yes) (on_board yes) (dnp no)
+    (property "Reference" "R12" (at 180.34 134.62 90)
+      (effects (font (size 1.27 1.27)))
+    )
+    (property "Value" "1k" (at 180.34 137.16 90)
+      (effects (font (size 1.27 1.27)))
+    )

Commit message: Add rest of footprints.
Parts:
- H1, H2, H3, H4: footprint (none) -> MountingHole:MountingHole_3.2mm_M3_Pad_Via
Changed lines of the file:
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@@
       (effects (font (size 1.27 1.27)) (justify left))
     )
-    (property "Footprint" "" (at 99.06 184.15 0)
+    (property "Footprint" "MountingHole:MountingHole_3.2mm_M3_Pad_Via" (at 99.06 184.15 0)
       (effects (font (size 1.27 1.27)) hide)
     )
@@
       (effects (font (size 1.27 1.27)) (justify left))
     )
-    (property "Footprint" "" (at 123.19 184.15 0)
+    (property "Footprint" "MountingHole:MountingHole_3.2mm_M3_Pad_Via" (at 123.19 184.15 0)
       (effects (font (size 1.27 1.27)) hide)
     )
@@
       (effects (font (size 1.27 1.27)) (justify left))
     )
-    (property "Footprint" "" (at 123.19 189.23 0)
+    (property "Footprint" "MountingHole:MountingHole_3.2mm_M3_Pad_Via" (at 123.19 189.23 0)
       (effects (font (size 1.27 1.27)) hide)
     )
@@
       (effects (font (size 1.27 1.27)) (justify left))
     )
-    (property "Footprint" "" (at 99.06 189.23 0)
-      (effects (font (size 1.27 1.27)) hide)
-    )
+    (property "Footprint" "MountingHole:MountingHole_3.2mm_M3_Pad_Via" (at 99.06 189.23 0)
+      (effects (font (size 1.27 1.27)) hide)
+    )

Commit message: PCB WIP.
Parts:
- J1, J10, J2: footprint TerminalBlock:TerminalBlock_Altech_AK300-2_P5.00mm -> TerminalBlock_Euroclamp:MVE252-5-V
- J3: renamed from J7; footprint TerminalBlock:TerminalBlock_Altech_AK300-2_P5.00mm -> TerminalBlock_Euroclamp:MVE252-5-V
- J4: renamed from J8; footprint TerminalBlock:TerminalBlock_Altech_AK300-2_P5.00mm -> TerminalBlock_Euroclamp:MVE252-5-V
- J5: renamed from J9; footprint TerminalBlock:TerminalBlock_Altech_AK300-2_P5.00mm -> TerminalBlock_Euroclamp:MVE252-5-V
- J9: renamed from J3; footprint TerminalBlock:TerminalBlock_Altech_AK300-2_P5.00mm -> TerminalBlock_Euroclamp:MVE252-5-V
Connections:
- net DCC/J1: now also J2.2 (Pin_2); no longer J2.1 (Pin_1)
- net DCC/J2: now also J2.1 (Pin_1); no longer J2.2 (Pin_2)
- net DCC/J3: now also J3.2 (Pin_2); no longer J3.1 (Pin_1)
- net DCC/J4: now also J3.1 (Pin_1); no longer J3.2 (Pin_2)
- net DCC/J5: now also J4.2 (Pin_2); no longer J4.1 (Pin_1)
- net DCC/J6: now also J4.1 (Pin_1); no longer J4.2 (Pin_2)
- net DCC/J7: now also J5.2 (Pin_2); no longer J5.1 (Pin_1)
- net DCC/J8: now also J5.1 (Pin_1); no longer J5.2 (Pin_2)
Other:
- moved on the sheet: J2, J3, J4, J5
Changed lines of the file:
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@@
     )
   )
-  (symbol (lib_id "Connector:Screw_Terminal_01x02") (at 29.21 60.96 0) (mirror y) (unit 1)
-    (in_bom yes) (on_board yes) (dnp no)
-    (property "Reference" "J8" (at 26.035 62.23 0)
-      (effects (font (size 1.27 1.27)))
-    )
-    (property "Value" "MVE252-5-V" (at 29.21 57.15 0)
-      (effects (font (size 1.27 1.27)) hide)
-    )
-    (property "Footprint" "TerminalBlock:TerminalBlock_Altech_AK300-2_P5.00mm" (at 29.21 60.96 0)
-      (effects (font (size 1.27 1.27)) hide)
-    )
-    (property "Datasheet" "~" (at 29.21 60.96 0)
-      (effects (font (size 1.27 1.27)) hide)
-    )
-    (pin "1")
-    (pin "2")
-    (instances
-      (project "railcomdet"
-        (path "/3e59d29f-2657-4552-9290-3c54fadfdf63"
-          (reference "J8") (unit 1)
+  (symbol (lib_id "Connector:Screw_Terminal_01x02") (at 29.21 63.5 180) (unit 1)
+    (in_bom yes) (on_board yes) (dnp no)
+    (property "Reference" "J4" (at 26.035 62.23 0)
+      (effects (font (size 1.27 1.27)))
+    )
+    (property "Value" "MVE252-5-V" (at 29.21 67.31 0)
+      (effects (font (size 1.27 1.27)) hide)
+    )
+    (property "Footprint" "TerminalBlock_Euroclamp:MVE252-5-V" (at 29.21 63.5 0)
+      (effects (font (size 1.27 1.27)) hide)
+    )
+    (property "Datasheet" "~" (at 29.21 63.5 0)
+      (effects (font (size 1.27 1.27)) hide)
+    )
+    (pin "1")
+    (pin "2")
+    (instances
+      (project "railcomdet"
+        (path "/3e59d29f-2657-4552-9290-3c54fadfdf63"
+          (reference "J4") (unit 1)
         )
       )
@@
       (effects (font (size 1.27 1.27)))
     )
-    (property "Footprint" "TerminalBlock:TerminalBlock_Altech_AK300-2_P5.00mm" (at 29.21 33.02 0)
+    (property "Footprint" "TerminalBlock_Euroclamp:MVE252-5-V" (at 29.21 33.02 0)
       (effects (font (size 1.27 1.27)) hide)
     )
@@
   (symbol (lib_id "Connector:Screw_Terminal_01x02") (at 270.51 31.115 0) (unit 1)
     (in_bom yes) (on_board yes) (dnp no)
-    (property "Reference" "J3" (at 273.685 32.385 0)
+    (property "Reference" "J9" (at 273.685 32.385 0)
       (effects (font (size 1.27 1.27)))
     )
@@
       (effects (font (size 1.27 1.27)))
     )
-    (property "Footprint" "TerminalBlock:TerminalBlock_Altech_AK300-2_P5.00mm" (at 270.51 31.115 0)
+    (property "Footprint" "TerminalBlock_Euroclamp:MVE252-5-V" (at 270.51 31.115 0)
       (effects (font (size 1.27 1.27)) hide)
     )
@@
       (project "railcomdet"
         (path "/3e59d29f-2657-4552-9290-3c54fadfdf63"
+          (reference "J9") (unit 1)
+        )
+      )
+    )
+  )
+  (symbol (lib_id "Device:C") (at 101.6 26.67 0) (unit 1)
+    (in_bom yes) (on_board yes) (dnp no) (fields_autoplaced)
+    (property "Reference" "C1" (at 105.41 25.4 0)
+      (effects (font (size 1.27 1.27)) (justify left))
+    )
+    (property "Value" "100n" (at 105.41 27.94 0)
+      (effects (font (size 1.27 1.27)) (justify left))
+    )
+    (property "Footprint" "Capacitor_SMD:C_0805_2012Metric" (at 102.5652 30.48 0)
+      (effects (font (size 1.27 1.27)) hide)
+    )
+    (property "Datasheet" "~" (at 101.6 26.67 0)
+      (effects (font (size 1.27 1.27)) hide)
+    )
+    (pin "1")
+    (pin "2")
+    (instances
+      (project "railcomdet"
+        (path "/3e59d29f-2657-4552-9290-3c54fadfdf63"
+          (reference "C1") (unit 1)
+        )
+      )
+    )
+  )
+  (symbol (lib_id "Connector:Screw_Terminal_01x02") (at 29.21 58.42 180) (unit 1)
+    (in_bom yes) (on_board yes) (dnp no)
+    (property "Reference" "J3" (at 26.035 57.15 0)
+      (effects (font (size 1.27 1.27)))
+    )
+    (property "Value" "MVE252-5-V" (at 29.21 62.23 0)
+      (effects (font (size 1.27 1.27)) hide)
+    )
+    (property "Footprint" "TerminalBlock_Euroclamp:MVE252-5-V" (at 29.21 58.42 0)
+      (effects (font (size 1.27 1.27)) hide)
+    )
+    (property "Datasheet" "~" (at 29.21 58.42 0)
+      (effects (font (size 1.27 1.27)) hide)
+    )
+    (pin "1")
+    (pin "2")
+    (instances
+      (project "railcomdet"
+        (path "/3e59d29f-2657-4552-9290-3c54fadfdf63"
           (reference "J3") (unit 1)
-        )
-      )
-    )
-  )
-  (symbol (lib_id "Device:C") (at 101.6 26.67 0) (unit 1)
-    (in_bom yes) (on_board yes) (dnp no) (fields_autoplaced)
-    (property "Reference" "C1" (at 105.41 25.4 0)
-      (effects (font (size 1.27 1.27)) (justify left))
-    )
-    (property "Value" "100n" (at 105.41 27.94 0)
-      (effects (font (size 1.27 1.27)) (justify left))
-    )
-    (property "Footprint" "Capacitor_SMD:C_0805_2012Metric" (at 102.5652 30.48 0)
-      (effects (font (size 1.27 1.27)) hide)
-    )
-    (property "Datasheet" "~" (at 101.6 26.67 0)
-      (effects (font (size 1.27 1.27)) hide)
-    )
-    (pin "1")
-    (pin "2")
-    (instances
-      (project "railcomdet"
-        (path "/3e59d29f-2657-4552-9290-3c54fadfdf63"
-          (reference "C1") (unit 1)
-        )
-      )
-    )
-  )
-  (symbol (lib_id "Connector:Screw_Terminal_01x02") (at 29.21 55.88 0) (mirror y) (unit 1)
-    (in_bom yes) (on_board yes) (dnp no)
-    (property "Reference" "J7" (at 26.035 57.15 0)
-      (effects (font (size 1.27 1.27)))
-    )
-    (property "Value" "MVE252-5-V" (at 29.21 52.07 0)
-      (effects (font (size 1.27 1.27)) hide)
-    )
-    (property "Footprint" "TerminalBlock:TerminalBlock_Altech_AK300-2_P5.00mm" (at 29.21 55.88 0)
-      (effects (font (size 1.27 1.27)) hide)
-    )
-    (property "Datasheet" "~" (at 29.21 55.88 0)
-      (effects (font (size 1.27 1.27)) hide)
-    )
-    (pin "1")
-    (pin "2")
-    (instances
-      (project "railcomdet"
-        (path "/3e59d29f-2657-4552-9290-3c54fadfdf63"
-          (reference "J7") (unit 1)
         )
       )
@@
       (effects (font (size 1.27 1.27)) hide)
     )
-    (property "Footprint" "TerminalBlock:TerminalBlock_Altech_AK300-2_P5.00mm" (at 270.51 36.195 0)
+    (property "Footprint" "TerminalBlock_Euroclamp:MVE252-5-V" (at 270.51 36.195 0)
       (effects (font (size 1.27 1.27)) hide)
     )
@@
     )
   )
-  (symbol (lib_id "Connector:Screw_Terminal_01x02") (at 29.21 66.04 0) (mirror y) (unit 1)
-    (in_bom yes) (on_board yes) (dnp no)
-    (property "Reference" "J9" (at 26.035 67.31 0)
-      (effects (font (size 1.27 1.27)))
-    )
-    (property "Value" "MVE252-5-V" (at 29.21 62.23 0)
-      (effects (font (size 1.27 1.27)) hide)
-    )
-    (property "Footprint" "TerminalBlock:TerminalBlock_Altech_AK300-2_P5.00mm" (at 29.21 66.04 0)
-      (effects (font (size 1.27 1.27)) hide)
-    )
-    (property "Datasheet" "~" (at 29.21 66.04 0)
-      (effects (font (size 1.27 1.27)) hide)
-    )
-    (pin "1")
-    (pin "2")
-    (instances
-      (project "railcomdet"
-        (path "/3e59d29f-2657-4552-9290-3c54fadfdf63"
-          (reference "J9") (unit 1)
+  (symbol (lib_id "Connector:Screw_Terminal_01x02") (at 29.21 68.58 180) (unit 1)
+    (in_bom yes) (on_board yes) (dnp no)
+    (property "Reference" "J5" (at 26.035 67.31 0)
+      (effects (font (size 1.27 1.27)))
+    )
+    (property "Value" "MVE252-5-V" (at 29.21 72.39 0)
+      (effects (font (size 1.27 1.27)) hide)
+    )
+    (property "Footprint" "TerminalBlock_Euroclamp:MVE252-5-V" (at 29.21 68.58 0)
+      (effects (font (size 1.27 1.27)) hide)
+    )
+    (property "Datasheet" "~" (at 29.21 68.58 0)
+      (effects (font (size 1.27 1.27)) hide)
+    )
+    (pin "1")
+    (pin "2")
+    (instances
+      (project "railcomdet"
+        (path "/3e59d29f-2657-4552-9290-3c54fadfdf63"
+          (reference "J5") (unit 1)
         )
       )
@@
     )
   )
-  (symbol (lib_id "Connector:Screw_Terminal_01x02") (at 29.21 50.8 0) (mirror y) (unit 1)
+  (symbol (lib_id "Connector:Screw_Terminal_01x02") (at 29.21 53.34 180) (unit 1)
     (in_bom yes) (on_board yes) (dnp no)
     (property "Reference" "J2" (at 26.035 52.07 0)
@@
       (effects (font (size 1.27 1.27)))
     )
-    (property "Footprint" "TerminalBlock:TerminalBlock_Altech_AK300-2_P5.00mm" (at 29.21 50.8 0)
-      (effects (font (size 1.27 1.27)) hide)
-    )
-    (property "Datasheet" "~" (at 29.21 50.8 0)
-      (effects (font (size 1.27 1.27)) hide)
-    )
+    (property "Footprint" "TerminalBlock_Euroclamp:MVE252-5-V" (at 29.21 53.34 0)
+      (effects (font (size 1.27 1.27)) hide)
+    )
+    (property "Datasheet" "~" (at 29.21 53.34 0)
+      (effects (font (size 1.27 1.27)) hide)
+    )
