File: pcb/mtb.kicad_sch (KiCad schematic)
At the start: 50 parts, among them J6 PINHEADER, J7 PINHEADER, J8 PROG/DEBUG, SW1 6x6, U12 STM32F103C8Tx, U13 AMS1117-3.3, U14 L78L05_SOT89, U15 SN75176AP, Y1 14,7456MHz

Commit message: Pcb tweaks.
Other:
- title: RailComDet - MTB part -> MTB-RC - MTBbus RailCom detector - MTB schematic
- moved on the sheet: D5, D6, R41, R42
Changed lines of the file:
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@@
   (paper "A4")
   (title_block
-    (title "RailComDet - MTB part")
+    (title "MTB-RC - MTBbus RailCom detector - MTB schematic")
     (date "2023-10-05")
+    (rev "see root")
     (company "Laboratory of railway vehicles control")
     (comment 1 "Kateřina Hanáková")
@@
   (junction (at 247.65 88.9) (diameter 0) (color 0 0 0 0)
   )
-  (junction (at 113.03 149.225) (diameter 0) (color 0 0 0 0)
-  )
   (junction (at 205.74 152.4) (diameter 0) (color 0 0 0 0)
   )
@@
   )
   (junction (at 252.73 27.94) (diameter 0) (color 0 0 0 0)
+  )
+  (junction (at 114.935 149.225) (diameter 0) (color 0 0 0 0)
   )
   (junction (at 270.51 144.78) (diameter 0) (color 0 0 0 0)
@@
     (stroke (width 0) (type default))
   )
-  (wire (pts (xy 113.03 149.225) (xy 113.03 151.765))
+  (wire (pts (xy 114.935 149.225) (xy 114.935 151.765))
     (stroke (width 0) (type default))
   )
@@
     (stroke (width 0) (type default))
   )
-  (wire (pts (xy 113.03 128.905) (xy 113.03 120.65))
+  (wire (pts (xy 114.935 128.905) (xy 114.935 120.65))
     (stroke (width 0) (type default))
   )
@@
     (stroke (width 0) (type default))
   )
-  (wire (pts (xy 120.65 149.225) (xy 113.03 149.225))
+  (wire (pts (xy 114.935 149.225) (xy 124.46 149.225))
     (stroke (width 0) (type default))
   )
@@
     (stroke (width 0) (type default))
   )
-  (wire (pts (xy 113.03 149.225) (xy 105.41 149.225))
+  (wire (pts (xy 105.41 149.225) (xy 114.935 149.225))
     (stroke (width 0) (type default))
   )
@@
     (stroke (width 0) (type default))
   )
-  (wire (pts (xy 86.36 118.11) (xy 120.65 118.11))
+  (wire (pts (xy 86.36 118.11) (xy 124.46 118.11))
     (stroke (width 0) (type default))
   )
@@
     (stroke (width 0) (type default))
   )
-  (wire (pts (xy 113.03 146.685) (xy 113.03 149.225))
+  (wire (pts (xy 114.935 146.685) (xy 114.935 149.225))
     (stroke (width 0) (type default))
   )
@@
     (stroke (width 0) (type default))
   )
-  (wire (pts (xy 113.03 136.525) (xy 113.03 139.065))
+  (wire (pts (xy 114.935 136.525) (xy 114.935 139.065))
     (stroke (width 0) (type default))
   )
@@
     (stroke (width 0) (type default))
   )
-  (wire (pts (xy 120.65 118.11) (xy 120.65 128.905))
+  (wire (pts (xy 124.46 118.11) (xy 124.46 128.905))
     (stroke (width 0) (type default))
   )
@@
     (stroke (width 0) (type default))
   )
-  (wire (pts (xy 120.65 136.525) (xy 120.65 139.065))
+  (wire (pts (xy 124.46 136.525) (xy 124.46 139.065))
     (stroke (width 0) (type default))
   )
@@
     (stroke (width 0) (type default))
   )
-  (wire (pts (xy 120.65 146.685) (xy 120.65 149.225))
+  (wire (pts (xy 124.46 146.685) (xy 124.46 149.225))
+    (stroke (width 0) (type default))
+  )
+  (wire (pts (xy 86.36 120.65) (xy 114.935 120.65))
     (stroke (width 0) (type default))
   )
   (wire (pts (xy 86.36 187.96) (xy 64.77 187.96))
-    (stroke (width 0) (type default))
-  )
-  (wire (pts (xy 86.36 120.65) (xy 113.03 120.65))
     (stroke (width 0) (type default))
   )
@@
     )
   )
-  (symbol (lib_id "Device:R") (at 113.03 132.715 0) (mirror y) (unit 1)
-    (in_bom yes) (on_board yes) (dnp no) (fields_autoplaced)
-    (property "Reference" "R41" (at 110.49 131.445 0)
-      (effects (font (size 1.27 1.27)) (justify left))
-    )
-    (property "Value" "1k" (at 110.49 133.985 0)
-      (effects (font (size 1.27 1.27)) (justify left))
-    )
-    (property "Footprint" "Resistor_SMD:R_0805_2012Metric_Pad1.20x1.40mm_HandSolder" (at 114.808 132.715 90)
-      (effects (font (size 1.27 1.27)) hide)
-    )
-    (property "Datasheet" "~" (at 113.03 132.715 0)
+  (symbol (lib_id "Device:R") (at 114.935 132.715 0) (mirror y) (unit 1)
+    (in_bom yes) (on_board yes) (dnp no)
+    (property "Reference" "R41" (at 113.03 131.445 0)
+      (effects (font (size 1.27 1.27)) (justify left))
+    )
+    (property "Value" "1k" (at 113.03 133.985 0)
+      (effects (font (size 1.27 1.27)) (justify left))
+    )
+    (property "Footprint" "Resistor_SMD:R_0805_2012Metric_Pad1.20x1.40mm_HandSolder" (at 116.713 132.715 90)
+      (effects (font (size 1.27 1.27)) hide)
+    )
+    (property "Datasheet" "~" (at 114.935 132.715 0)
       (effects (font (size 1.27 1.27)) hide)
     )
@@
     )
   )
-  (symbol (lib_id "Device:LED") (at 113.03 142.875 270) (mirror x) (unit 1)
-    (in_bom yes) (on_board yes) (dnp no)
-    (property "Reference" "D5" (at 111.76 140.335 0)
-      (effects (font (size 1.27 1.27)))
-    )
-    (property "Value" "GREEN" (at 115.57 142.875 0)
-      (effects (font (size 1.27 1.27)))
-    )
-    (property "Footprint" "LED_SMD:LED_0805_2012Metric_Pad1.15x1.40mm_HandSolder" (at 113.03 142.875 0)
-      (effects (font (size 1.27 1.27)) hide)
-    )
-    (property "Datasheet" "~" (at 113.03 142.875 0)
+  (symbol (lib_id "Device:LED") (at 114.935 142.875 270) (mirror x) (unit 1)
+    (in_bom yes) (on_board yes) (dnp no)
+    (property "Reference" "D5" (at 112.395 142.875 0)
+      (effects (font (size 1.27 1.27)))
+    )
+    (property "Value" "GREEN" (at 117.475 142.875 0)
+      (effects (font (size 1.27 1.27)))
+    )
+    (property "Footprint" "LED_SMD:LED_0805_2012Metric_Pad1.15x1.40mm_HandSolder" (at 114.935 142.875 0)
+      (effects (font (size 1.27 1.27)) hide)
+    )
+    (property "Datasheet" "~" (at 114.935 142.875 0)
       (effects (font (size 1.27 1.27)) hide)
     )
@@
     )
   )
-  (symbol (lib_id "Device:LED") (at 120.65 142.875 270) (mirror x) (unit 1)
-    (in_bom yes) (on_board yes) (dnp no)
-    (property "Reference" "D6" (at 119.38 140.335 0)
-      (effects (font (size 1.27 1.27)))
-    )
-    (property "Value" "RED" (at 123.19 142.875 0)
-      (effects (font (size 1.27 1.27)))
-    )
-    (property "Footprint" "LED_SMD:LED_0805_2012Metric_Pad1.15x1.40mm_HandSolder" (at 120.65 142.875 0)
-      (effects (font (size 1.27 1.27)) hide)
-    )
-    (property "Datasheet" "~" (at 120.65 142.875 0)
+  (symbol (lib_id "Device:LED") (at 124.46 142.875 270) (mirror x) (unit 1)
+    (in_bom yes) (on_board yes) (dnp no)
+    (property "Reference" "D6" (at 121.92 142.875 0)
+      (effects (font (size 1.27 1.27)))
+    )
+    (property "Value" "RED" (at 127 142.875 0)
+      (effects (font (size 1.27 1.27)))
+    )
+    (property "Footprint" "LED_SMD:LED_0805_2012Metric_Pad1.15x1.40mm_HandSolder" (at 124.46 142.875 0)
+      (effects (font (size 1.27 1.27)) hide)
+    )
+    (property "Datasheet" "~" (at 124.46 142.875 0)
       (effects (font (size 1.27 1.27)) hide)
     )
@@
   )
   (symbol (lib_id "Device:R") (at 105.41 132.715 0) (mirror y) (unit 1)
-    (in_bom yes) (on_board yes) (dnp no) (fields_autoplaced)
-    (property "Reference" "R39" (at 102.87 131.445 0)
-      (effects (font (size 1.27 1.27)) (justify left))
-    )
-    (property "Value" "1k" (at 102.87 133.985 0)
+    (in_bom yes) (on_board yes) (dnp no)
+    (property "Reference" "R39" (at 103.505 131.445 0)
+      (effects (font (size 1.27 1.27)) (justify left))
+    )
+    (property "Value" "1k" (at 103.505 133.985 0)
       (effects (font (size 1.27 1.27)) (justify left))
     )
@@
     )
   )
-  (symbol (lib_id "Device:R") (at 120.65 132.715 0) (mirror y) (unit 1)
-    (in_bom yes) (on_board yes) (dnp no) (fields_autoplaced)
-    (property "Reference" "R42" (at 118.11 131.445 0)
-      (effects (font (size 1.27 1.27)) (justify left))
-    )
-    (property "Value" "1k" (at 118.11 133.985 0)
-      (effects (font (size 1.27 1.27)) (justify left))
-    )
-    (property "Footprint" "Resistor_SMD:R_0805_2012Metric_Pad1.20x1.40mm_HandSolder" (at 122.428 132.715 90)
-      (effects (font (size 1.27 1.27)) hide)
-    )
-    (property "Datasheet" "~" (at 120.65 132.715 0)
+  (symbol (lib_id "Device:R") (at 124.46 132.715 0) (mirror y) (unit 1)
+    (in_bom yes) (on_board yes) (dnp no)
+    (property "Reference" "R42" (at 122.555 131.445 0)
+      (effects (font (size 1.27 1.27)) (justify left))
+    )
+    (property "Value" "1k" (at 122.555 133.985 0)
+      (effects (font (size 1.27 1.27)) (justify left))
+    )
+    (property "Footprint" "Resistor_SMD:R_0805_2012Metric_Pad1.20x1.40mm_HandSolder" (at 126.238 132.715 90)
+      (effects (font (size 1.27 1.27)) hide)
+    )
+    (property "Datasheet" "~" (at 124.46 132.715 0)
       (effects (font (size 1.27 1.27)) hide)
     )
@@
   (symbol (lib_id "Device:LED") (at 105.41 142.875 270) (mirror x) (unit 1)
     (in_bom yes) (on_board yes) (dnp no)
-    (property "Reference" "D4" (at 104.14 140.335 0)
+    (property "Reference" "D4" (at 102.87 142.875 0)
       (effects (font (size 1.27 1.27)))
     )
@@
     )
   )
-  (symbol (lib_id "power:GND") (at 113.03 151.765 0) (mirror y) (unit 1)
+  (symbol (lib_id "power:GND") (at 114.935 151.765 0) (mirror y) (unit 1)
     (in_bom yes) (on_board yes) (dnp no) (fields_autoplaced)
-    (property "Reference" "#PWR049" (at 113.03 158.115 0)
-      (effects (font (size 1.27 1.27)) hide)
-    )
-    (property "Value" "GND" (at 113.03 156.845 0)
-      (effects (font (size 1.27 1.27)))
-    )
-    (property "Footprint" "" (at 113.03 151.765 0)
-      (effects (font (size 1.27 1.27)) hide)
-    )
-    (property "Datasheet" "" (at 113.03 151.765 0)
-      (effects (font (size 1.27 1.27)) hide)
-    )
+    (property "Reference" "#PWR049" (at 114.935 158.115 0)
+      (effects (font (size 1.27 1.27)) hide)
+    )
+    (property "Value" "GND" (at 114.935 156.845 0)
+      (effects (font (size 1.27 1.27)))
+    )
+    (property "Footprint" "" (at 114.935 151.765 0)
+      (effects (font (size 1.27 1.27)) hide)
+    )
+    (property "Datasheet" "" (at 114.935 151.765 0)
+      (effects (font (size 1.27 1.27)) hide)
+    )
